File: V1/TempWatchtV1.kicad_pcb (KiCad board)
At the start: 4 copper layers, 70 x 35 mm, 65 parts, among them CN1 SM03B-SRSS-TB(LF)(SN)(P), CN10 SM04B-SRSS-TB (LF)(SN), CN11 SM02B-PASS-1-TBT(LF)(SN), CN2 SM03B-SRSS-TB(LF)(SN)(P), CN3 SM03B-SRSS-TB(LF)(SN)(P), CN4 SM03B-SRSS-TB(LF)(SN)(P), CN5 SM03B-SRSS-TB(LF)(SN)(P), CN6 SM03B-SRSS-TB(LF)(SN)(P), CN7 SM03B-SRSS-TB(LF)(SN)(P), CN8 SM03B-SRSS-TB(LF)(SN)(P)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

Commit message: Latest
Parts:
- removed U4: ESP32-S3-WROOM-1(N8R2), easyeda2kicad:WIRELM-SMD_ESP32-S3-WROOM-1
- added U3: ESP32-S3-WROOM-1U-N8R2, easyeda2kicad:WIRELM-SMD_ESP32-S3-WROOM-1U, F.Cu at (131.8, 114.7)
